File: onboarding.kicad_sch (KiCad schematic)
At the start: 46 parts, among them J1 USB_C_Receptacle_USB2.0_16P, J2 Conn_01x04, J3 Conn_02x03_Odd_Even, J4 530470260, SW1 RESET, SW2 BOOT, U1 LM1117DT-3.3, U2 ASM330LHHXTR, U3 VL53L0CXV0DH_1, U4 USBLC6-2SC6, U5 ESP32-S3-WROOM-1, U6 MLX90614ESF-BCF-000-TU, U7 MLX90641ESF-BCB-000-TU, U8 TJA1462ATK_0Z

Commit message: Buck Converter added
Parts:
- added C15: 100nF, Capacitor_SMD:C_0402_1005Metric_Pad0.74x0.62mm_HandSolder, symbol Device:C_Small
- added C16, C17: 10uF, Capacitor_SMD:C_0603_1608Metric, symbol Device:C_Small
- added C18: 4U7, Capacitor_SMD:C_0603_1608Metric, symbol Device:C_Small
- added L2: NRS5030T3R3MMGJ, sensors:IND_NRS5030T3R3MMGJ_TAY-M, symbol 2026-08-19_19-38-41:NRS5030T3R3MMGJ
- added R17, R18: 100R, Resistor_SMD:R_0603_1608Metric_Pad0.98x0.95mm_HandSolder, symbol Device:R_Small
- added R19: 13K7, Resistor_SMD:R_0402_1005Metric_Pad0.72x0.64mm_HandSolder, symbol Device:R_Small
- added U11: STEF12SAGR, sensors:IC8_STEF12SAGR_STM, symbol 2026-08-19_18-54-03:STEF12SAGR
- added U12: LMR51420YFDDCR, sensors:IC8_STEF12SAGR_STM, symbol LMR51420YFDDCR:LMR51420YFDDCR
- renumbered C11 to C10, C12 to C11, C13 to C12, C14 to C13, C4 to C3, C5 to C4, C6 to C5, C7 to C6, C8 to C7, C9 to C8, C10 to C9, D3 to D2, D4 to D3, D5 to D4
Connections:
- net +5V: now also C6.1, U4.5 (VBUS), L2.2
- net GND: now also C16.2, C17.2, C18.2, R19.1, U11.4 (GND), U12.1 (GND)
- new net: R18.1, R19.2, U12.4 (FB)
- new net: C15.1, U12.6 (CB)
- new net: C15.2, L2.1, U12.2 (SW)
- new net: C16.1, C17.1, R18.2
- new net: R17.2, U11.1 (ILim)
- new net 12 V POST FUSE: C18.1, R17.1, U11.5 (Source), U11.6 (Source), U12.3 (VIN), U12.5 (EN)
- no-connect marks 22 -> 26
Other:
- note added: "12v -> 5v"
- moved on the sheet: J4, R15, U8

Commit message: finished circuit schematic
Parts:
- removed J4: 530470260, sensors:CONN02_530470260_MOL, symbol 530470260:530470260
- added J2, J3: 430450800, sensors:CONN_SD-43045-001_08_MOL, symbol 430450800:430450800
- added J6, J7: 430451600, sensors:CONN_SD-43045-001_16_MOL, symbol 430451600:430451600
- U7: renamed from U12; footprint sensors:IC8_STEF12SAGR_STM -> sensors:SOT95P280X110-6N
- renumbered C18 to C11, C15 to C12, C16 to C13, C17 to C14, C11 to C15, C12 to C16, C13 to C17, J2 to J4, J3 to J5, L2 to L1, R9 to R10, R10 to R11, R11 to R12, R12 to R13, R13 to R14, R14 to R15, R19 to R16, R15 to R17, R17 to R6, R6 to R7, R7 to R8, R8 to R9, U8 to U10, U11 to U5, U5 to U6, U6 to U8, U7 to U9
Connections:
- net +3V3: now also J6.1, J6.2, J7.1, J7.2
- net 12 V POST FUSE: no longer R6.1
- net BRAKE_PWM: now also J6.15, J6.16, J7.15, J7.16
- net GND: now also J2.3, J2.4, J3.3, J3.4, J6.3, J6.4, J7.3, J7.4
- net SCL: now also J6.7, J6.8, J7.7, J7.8
- net SCL2_TTS: now also J6.10, J6.9, J7.10, J7.9
- net SDA: now also J6.5, J6.6, J7.5, J7.6
- net SDA2_TTS: now also J6.11, J6.12, J7.11, J7.12
- net CANL: now reaches R17.1, U10.6 (CANL)
- net CANL: now also J2.5, J2.6, J3.5, J3.6
- net CANH: now reaches R17.2, U10.7 (CANH)
- net CANH: now also J2.7, J2.8, J3.7, J3.8
- new net +12V: J2.1, J2.2, J3.1, J3.2, R6.1
- new net BRAKE_SCL: J6.13, J6.14, J7.13, J7.14
Other:
- note added: "Power & CAN Conector"
