File: onboarding.kicad_sch (KiCad schematic)
At the start: 62 parts, among them J1 USB_C_Receptacle_USB2.0_16P, J10 430450400, J2 430450800, J3 Conn_01x04, J4 Conn_02x03_Odd_Even, J5 430450400, J6 430450400, J7 430450400, J8 430450400, J9 430450400, SW1 RESET, SW2 BOOT, U1 LM1117DT-3.3, U10 TJA1462ATK_0Z, U2 ASM330LHHXTR, U3 VL53L0CXV0DH_1, U4 USBLC6-2SC6, U5 STEF12SAGR, U6 ESP32-S3-WROOM-1, U7 LMR51420YFDDCR, U8 MLX90614ESF-BCF-000-TU, U9 MLX90641ESF-BCB-000-TU

Commit message: Almost
Parts:
- J1: footprint Connector_USB:USB_C_Receptacle_HRO_TYPE-C-31-M-12 -> Connector_USB:USB_C_Receptacle_Palconn_UTC16-G
Changed lines of the file:
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@@
 			)
 		)
-		(property "Footprint" "Connector_USB:USB_C_Receptacle_HRO_TYPE-C-31-M-12"
+		(property "Footprint" "Connector_USB:USB_C_Receptacle_Palconn_UTC16-G"
 			(at 40.64 38.1 0)
 			(hide yes)
