File: onboarding.kicad_pcb (KiCad board)
At the start: 4 copper layers, 50 x 50 mm, 54 parts, among them J1 USB_C_Receptacle_USB2.0_16P, J2 Conn_01x04, J3 Conn_02x03_Odd_Even, J4 530470260, SW1 RESET, SW2 BOOT, U1 LM1117DT-3.3, U2 ASM330LHHXTR, U3 VL53L0CXV0DH_1, U4 USBLC6-2SC6, U5 ESP32-S3-WROOM-1, U6 MLX90614ESF-BCF-000-TU, U7 MLX90641ESF-BCB-000-TU, U8 TJA1462ATK_0Z

Commit message: Buck Converter added
Parts:
- removed C3: 10nF, Capacitor_SMD:C_0402_1005Metric
- removed D2: 1N5817, Diode_SMD:D_SOD-123
- removed F1: Polyfuse 1A, Fuse:Fuse_1206_3216Metric
- removed FB1: BLM21PG220, Inductor_SMD:L_0805_2012Metric
- moved R12 57.5 mm to (213.1, 136.0)
- moved R13 57.5 mm to (202.1, 128.3)
- moved U2 57.5 mm to (208.0, 132.3)
- moved C13 57.5 mm to (202.6, 146.1)
- moved C14 57.5 mm to (221.1, 151.7)
- moved C6 57.5 mm to (199.9, 136.9)
- moved D3 57.5 mm to (216.3, 130.5)
- moved R10 57.5 mm to (204.9, 128.2)
- moved R11 57.5 mm to (211.1, 136.0)
- moved R7 57.5 mm to (219.7, 131.6)
- moved R8 57.5 mm to (219.9, 129.8)
- moved U3 57.5 mm to (201.9, 135.0)
- moved U6 57.5 mm to (221.0, 141.5)
- moved U7 57.5 mm to (208.5, 144.8)
- moved C12 57.5 mm to (202.0, 149.7)
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Connections:
- C7 pad 1: Net-(U4-VBUS) -> +5V
- J1 pad A4: Net-(U4-VBUS) -> unconnected-(J1-VBUS-PadA4)_3
- J1 pad A9: Net-(U4-VBUS) -> unconnected-(J1-VBUS-PadA4)
- J1 pad B4: Net-(U4-VBUS) -> unconnected-(J1-VBUS-PadA4)_1
- J1 pad B9: Net-(U4-VBUS) -> unconnected-(J1-VBUS-PadA4)_2
- U4 pad 5: Net-(U4-VBUS) -> +5V
Routing:
- net +5V: track 96.2 -> 0.00 mm, vias 2 -> 0
- net +3V3: track 87.9 -> 0.00 mm, vias 14 -> 0
- net GND: track 69.3 -> 0.00 mm, vias 35 -> 0
- net /ESP_EN: track 62.3 -> 0.00 mm, vias 3 -> 0
- net /SDA: track 48.9 -> 0.00 mm, vias 4 -> 0
- net /SCL: track 40.2 -> 0.00 mm, vias 2 -> 0
- net /ESP_IO0: track 36.0 -> 0.00 mm
- net /SDA2_TTS: track 30.8 -> 0.00 mm, vias 2 -> 0
- net /SCL2_TTS: track 26.4 -> 0.00 mm, vias 2 -> 0
- net /IO5: track 26.3 -> 0.00 mm, vias 2 -> 0
- net /BRAKE_SCL_DBG: track 25.8 -> 0.00 mm, vias 2 -> 0
- net /IO4: track 25.6 -> 0.00 mm, vias 2 -> 0
- net /FDCAN_TX: track 25.2 -> 0.00 mm, vias 2 -> 0
- net /G_RGB: track 23.7 -> 0.00 mm, vias 2 -> 0
- net /BRAKE_PWM: track 22.5 -> 0.00 mm, vias 2 -> 0
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Other:
- outline, holes or cut-outs redrawn

Commit message: finished circuit schematic
Parts:
- added C14: 100nF, Capacitor_SMD:C_0402_1005Metric_Pad0.74x0.62mm_HandSolder, F.Cu at (114.8, 146.8)
- added C15: 100nF, Capacitor_SMD:C_0402_1005Metric_Pad0.74x0.62mm_HandSolder, F.Cu at (106.1, 159.0)
- added C16: 10uF, Capacitor_SMD:C_0603_1608Metric, F.Cu at (106.5, 149.8)
- added C17: 10uF, Capacitor_SMD:C_0603_1608Metric, F.Cu at (106.5, 152.3)
- added C18: 4U7, Capacitor_SMD:C_0603_1608Metric, F.Cu at (106.5, 154.8)
- added L1: NRS5030T3R3MMGJ, sensors:IND_NRS5030T3R3MMGJ_TAY-M, F.Cu at (112.7, 139.6)
- added L2: NRS5030T3R3MMGJ, sensors:IND_NRS5030T3R3MMGJ_TAY-M, F.Cu at (113.2, 152.1)
- added R16: 100R, Resistor_SMD:R_0603_1608Metric_Pad0.98x0.95mm_HandSolder, F.Cu at (115.3, 144.5)
- added R17: 100R, Resistor_SMD:R_0603_1608Metric_Pad0.98x0.95mm_HandSolder, F.Cu at (110.7, 157.0)
- added R18: 100R, Resistor_SMD:R_0603_1608Metric_Pad0.98x0.95mm_HandSolder, F.Cu at (110.7, 159.5)
- added R19: 13K7, Resistor_SMD:R_0402_1005Metric_Pad0.72x0.64mm_HandSolder, F.Cu at (106.1, 157.0)
- added U11: STEF12SAGR, sensors:IC8_STEF12SAGR_STM, F.Cu at (115.4, 158.0)
- added U12: LMR51420YFDDCR, sensors:SOT95P280X110-6N, F.Cu at (94.1, 154.8)
- added U9: STEF12SAGR, sensors:IC8_STEF12SAGR_STM, F.Cu at (110.6, 145.5)
- moved J1 26.6 mm to (144.0, 89.5)
- renumbered C11 to C10, C12 to C11, C13 to C12, C14 to C13, C4 to C3, C5 to C4, C6 to C5, C7 to C6, C8 to C7, C9 to C8, C10 to C9, D3 to D2, D4 to D3, D5 to D4

Commit message: Maybe I can get this done
Parts:
- removed C18: 4U7, Capacitor_SMD:C_0603_1608Metric
- removed H1, H2, H3, H4: MountingHole, MountingHole:MountingHole_3.2mm_M3
- removed J3: Conn_02x03_Odd_Even, Connector_PinHeader_2.54mm:PinHeader_2x03_P2.54mm_Vertical
- removed L2: NRS5030T3R3MMGJ, sensors:IND_NRS5030T3R3MMGJ_TAY-M
- removed R19: 13K7, Resistor_SMD:R_0402_1005Metric_Pad0.72x0.64mm_HandSolder
- removed U11: STEF12SAGR, sensors:IC8_STEF12SAGR_STM
- removed U12: LMR51420YFDDCR, sensors:SOT95P280X110-6N
- added J11: 430450800, sensors:CONN_SD-43045-001_08_MOL, F.Cu at (170.9, 55.4)
- added J12: 430450800, sensors:CONN_SD-43045-001_08_MOL, F.Cu at (170.9, 69.3)
- added J13: 430450800, sensors:CONN_SD-43045-001_08_MOL, F.Cu at (165.0, 85.5)
- added J14: 430450800, sensors:CONN_SD-43045-001_08_MOL, F.Cu at (130.2, 41.3)
- added J15: 430450800, sensors:CONN_SD-43045-001_08_MOL, F.Cu at (129.2, 59.6)
- added J16: 430450800, sensors:CONN_SD-43045-001_08_MOL, F.Cu at (128.7, 78.1)
- added J5: Conn_02x03_Odd_Even, Connector_PinHeader_2.54mm:PinHeader_2x03_P2.54mm_Vertical, F.Cu at (68.4, 86.0)
- added U10: TJA1462ATK_0Z, sensors:SON65P300X300X100-9N, F.Cu at (121.0, 90.0)
- C11: value 100nF -> 4U7; footprint Capacitor_SMD:C_0402_1005Metric_Pad0.74x0.62mm_HandSolder -> Capacitor_SMD:C_0603_1608Metric
- C12, C17: value 10uF -> 100nF; footprint Capacitor_SMD:C_0603_1608Metric -> Capacitor_SMD:C_0402_1005Metric_Pad0.74x0.62mm_HandSolder
- C13, C14: value 100nF -> 10uF; footprint Capacitor_SMD:C_0402_1005Metric_Pad0.74x0.62mm_HandSolder -> Capacitor_SMD:C_0603_1608Metric
- J1: footprint Connector_USB:USB_C_Receptacle_GCT_USB4105-xx-A_16P_TopMnt_Horizontal -> Connector_USB:USB_C_Receptacle_HCTL_HC-TYPE-C-16P-01A
- J2: value Conn_01x04 -> 430450800; footprint Connector_JST:JST_SH_SM04B-SRSS-TB_1x04-1MP_P1.00mm_Horizontal -> sensors:CONN_SD-43045-001_08_MOL
- J4: value 530470260 -> Conn_01x04; footprint sensors:CONN02_530470260_MOL -> Connector_JST:JST_SH_SM04B-SRSS-TB_1x04-1MP_P1.00mm_Horizontal
- R13: value 1K -> 4K7
- R14: value 10K -> 1K
- R15: value 100R -> 10K; footprint Resistor_SMD:R_0603_1608Metric_Pad0.98x0.95mm_HandSolder -> Resistor_SMD:R_0402_1005Metric_Pad0.72x0.64mm_HandSolder
- R16: value 100R -> 13K7; footprint Resistor_SMD:R_0603_1608Metric_Pad0.98x0.95mm_HandSolder -> Resistor_SMD:R_0402_1005Metric_Pad0.72x0.64mm_HandSolder
- R6: value 1K -> 100R; footprint Resistor_SMD:R_0402_1005Metric_Pad0.72x0.64mm_HandSolder -> Resistor_SMD:R_0603_1608Metric_Pad0.98x0.95mm_HandSolder
- R9: value 4K7 -> 1K
- U5: value ESP32-S3-WROOM-1 -> STEF12SAGR; footprint RF_Module:ESP32-S3-WROOM-1 -> sensors:IC8_STEF12SAGR_STM
- U6: value MLX90614ESF-BCF-000-TU -> ESP32-S3-WROOM-1; footprint sensors:MLX90614xCF_MEL -> RF_Module:ESP32-S3-WROOM-1
- U7: value MLX90641ESF-BCB-000-TU -> LMR51420YFDDCR; footprint sensors:TO254P912H435-4 -> sensors:SOT95P280X110-6N
- U8: value TJA1462ATK_0Z -> MLX90614ESF-BCF-000-TU; footprint sensors:SON65P300X300X100-9N -> sensors:MLX90614xCF_MEL
- U9: value STEF12SAGR -> MLX90641ESF-BCB-000-TU; footprint sensors:IC8_STEF12SAGR_STM -> sensors:MLX90614xCF_MEL
- moved R5 176.7 mm to (73.0, 44.6)
- moved R15 176.6 mm to (75.5, 46.0), turned to 0 degrees
- moved C8 175.4 mm to (73.8, 41.5), turned to 0 degrees
- moved D3 171.6 mm to (77.0, 41.5), turned to 0 degrees
- moved R7 164.4 mm to (74.5, 54.5), turned to -90 degrees
- moved D2 161.3 mm to (76.0, 51.0)
- moved R8 160.3 mm to (79.4, 52.5)
- moved J4 158.0 mm to (70.0, 92.8), turned to -90 degrees
- moved SW1 156.2 mm to (69.0, 41.5), turned to 0 degrees
- moved SW2 153.0 mm to (68.8, 48.0), turned to 0 degrees
- moved U6 151.3 mm to (102.2, 47.8)
- moved D4 146.2 mm to (72.6, 48.0), turned to 0 degrees
- moved R11 135.1 mm to (97.5, 62.9)
- moved R12 134.6 mm to (100.0, 63.0)
- moved R10 134.5 mm to (91.1, 56.5), turned to 0 degrees
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Connections:
- C11 pad 1: +3V3 -> +12V
- C12 pad 1: +3V3 -> Net-(U7-CB)
- C12 pad 2: GND -> Net-(U7-SW)
- C13 pad 1: +3V3 -> Net-(C13-Pad1)
- C14 pad 1: Net-(U10-CB) -> Net-(C13-Pad1)
- C14 pad 2: Net-(U10-SW) -> GND
- C15 pad 1: Net-(U12-CB) -> +3V3
- C15 pad 2: Net-(U12-SW) -> GND
- C16 pad 1: Net-(C16-Pad1) -> +3V3
- C17 pad 1: Net-(C16-Pad1) -> +3V3
- J2 pad 1: GND -> +12V
- J2 pad 2: +3V3 -> +12V
- J2 pad 3: /SDA -> GND
- J2 pad 4: /SCL -> GND
- J4 pad 1: Net-(U8-CANH) -> GND
- J4 pad 2: Net-(U8-CANL) -> +3V3
- L1 pad 1: +5V -> Net-(U7-SW)
- L1 pad 2: Net-(U10-SW) -> +5V
- R10 pad 2: /SLC -> /SDA
- R11 pad 1: /SCL2_TTS -> +3V3
- R11 pad 2: +3V3 -> /SCL
- R12 pad 1: /SDA2_TTS -> +3V3
- R12 pad 2: +3V3 -> /SCL2_TTS
- R13 pad 1: Net-(U5-IO3) -> +3V3
- R13 pad 2: +3V3 -> /SDA2_TTS
- R14 pad 1: /ESP_IO0 -> Net-(U6-IO3)
- R14 pad 2: Net-(D4-A2) -> +3V3
- R15 pad 1: Net-(U8-CANL) -> /ESP_IO0
- R15 pad 2: Net-(U8-CANH) -> Net-(D4-A2)
- R16 pad 1: unconnected-(R16-Pad1) -> GND
- R16 pad 2: Net-(U9-ILim) -> Net-(U7-FB)
- R17 pad 1: /12 V POST FUSE -> /CANL
- R17 pad 2: Net-(U11-ILim) -> /CANH
- R18 pad 1: Net-(U12-FB) -> Net-(U7-FB)
- R18 pad 2: Net-(C16-Pad1) -> Net-(C13-Pad1)
- R6 pad 1: Net-(D2-RK) -> +12V
- R6 pad 2: /R_RGB -> Net-(U5-ILim)
- R7 pad 1: Net-(D2-GK) -> Net-(D2-RK)
- R7 pad 2: /G_RGB -> /R_RGB
- R8 pad 1: Net-(D2-BK) -> Net-(D2-GK)
- R8 pad 2: /B_RGB -> /G_RGB
- R9 pad 1: +3V3 -> Net-(D2-BK)
- R9 pad 2: /SDA -> /B_RGB
- U4 pad 1: /USB_D- -> /USB_D+
- U4 pad 3: /USB_D+ -> /USB_D-
- U4 pad 4: /D+ -> /D-
- U4 pad 6: /D- -> /D+
- U5 pad 1: GND -> Net-(U5-ILim)
- U5 pad 2: +3V3 -> unconnected-(U5-En/Fault-Pad2)
- U5 pad 3: /ESP_EN -> unconnected-(U5-dV/dt-Pad3)
- U5 pad 4: /IO4 -> GND
- U5 pad 5: /IO5 -> +12V
- U5 pad 6: unconnected-(U5-IO6-Pad6) -> +12V
- U6 pad 1: /BRAKE_SCL_DBG -> GND
- U6 pad 2: /BRAKE_PWM -> +3V3
- U6 pad 3: +3V3 -> /ESP_EN
- U6 pad 4: GND -> /IO4
- U7 pad 1: /SDA2_TTS -> GND
- U7 pad 2: +3V3 -> Net-(U7-SW)
- U7 pad 3: GND -> +12V
- U7 pad 4: /SCL2_TTS -> Net-(U7-FB)
- U8 pad 1: /FDCAN_RX -> /BRAKE_SCL
- U8 pad 2: GND -> /BRAKE_PWM
- U8 pad 3: +5V -> +3V3
- U8 pad 4: /FDCAN_TX -> GND
- U9 pad 1: Net-(U9-ILim) -> /SDA2_TTS
- U9 pad 2: unconnected-(U9-En/Fault-Pad2) -> +3V3
- U9 pad 3: unconnected-(U9-dV/dt-Pad3) -> GND
- U9 pad 4: GND -> /SCL2_TTS
Routing:
- net GND: track 0.00 -> 122.0 mm, vias 0 -> 31
- net /SCL: track 0.00 -> 110.2 mm, vias 0 -> 2
- net /SDA: track 0.00 -> 107.2 mm, vias 0 -> 4
- net /ESP_IO0: track 0.00 -> 103.9 mm
- net +5V: track 0.00 -> 100.7 mm, vias 0 -> 3
- net +3V3: track 0.00 -> 81.4 mm, vias 0 -> 15
- net /FDCAN_TX: track 0.00 -> 72.9 mm, vias 0 -> 2
- net /FDCAN_RX: track 0.00 -> 63.5 mm
- net /ESP_TXD: track 0.00 -> 62.7 mm, vias 0 -> 2
- net /ESP_RXD: track 0.00 -> 57.3 mm, vias 0 -> 2
- net /B_RGB: track 0.00 -> 54.2 mm, vias 0 -> 2
- net /R_RGB: track 0.00 -> 52.3 mm, vias 0 -> 2
- net /BRAKE_PWM: track 0.00 -> 51.1 mm
- net /IO5: track 0.00 -> 42.3 mm, vias 0 -> 4
- net /G_RGB: track 0.00 -> 40.3 mm, vias 0 -> 2
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Other:
- board size 50 x 50 mm -> 75 x 75 mm

Commit message: The end is inevitable
Parts:
- removed J11, J12, J13, J14, J15, J16: 430450800, sensors:CONN_SD-43045-001_08_MOL
- added J10: 430450400, sensors:CONN_SD-43045-001_04_MOL, F.Cu at (211.1, 123.6)
- added J3: Conn_01x04, Connector_JST:JST_SH_SM04B-SRSS-TB_1x04-1MP_P1.00mm_Horizontal, F.Cu at (23.0, 180.0)
- added J6: 430450400, sensors:CONN_SD-43045-001_04_MOL, F.Cu at (158.5, 123.6)
- added J7: 430450400, sensors:CONN_SD-43045-001_04_MOL, F.Cu at (59.0, 157.8)
- added J8: 430450400, sensors:CONN_SD-43045-001_04_MOL, F.Cu at (59.6, 143.4)
- added J9: 430450400, sensors:CONN_SD-43045-001_04_MOL, F.Cu at (197.9, 123.6)
- J1: footprint Connector_USB:USB_C_Receptacle_HCTL_HC-TYPE-C-16P-01A -> Connector_USB:USB_C_Receptacle_HRO_TYPE-C-31-M-12
- J4: value Conn_01x04 -> Conn_02x03_Odd_Even; footprint Connector_JST:JST_SH_SM04B-SRSS-TB_1x04-1MP_P1.00mm_Horizontal -> Connector_PinHeader_2.54mm:PinHeader_2x03_P2.54mm_Vertical
- J5: value Conn_02x03_Odd_Even -> 430450400; footprint Connector_PinHeader_2.54mm:PinHeader_2x03_P2.54mm_Vertical -> sensors:CONN_SD-43045-001_04_MOL
- moved C6 179.8 mm to (30.9, 148.5)
- moved D3 146.5 mm to (43.9, 184.2), turned to -90 degrees
- moved SW1 144.8 mm to (40.7, 183.5)
- moved C8 144.5 mm to (46.6, 183.4), turned to 90 degrees
- moved R5 141.8 mm to (45.1, 183.6), turned to -90 degrees
- moved R11 112.0 mm to (38.6, 158.2)
- moved R12 111.9 mm to (41.2, 158.2)
- moved R10 111.8 mm to (31.0, 150.8)
- moved R13 111.8 mm to (43.2, 158.0)
- moved R14 111.6 mm to (36.2, 157.1)
- moved C3 111.5 mm to (43.3, 166.8)
- moved U6 111.3 mm to (43.2, 142.1)
- moved D1 110.3 mm to (59.0, 184.0)
- moved C9 110.2 mm to (28.9, 138.1)
- moved U10 110.1 mm to (52.2, 176.0), turned to 0 degrees
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Connections:
- J4 pad 1: GND -> /ESP_EN
- J4 pad 3: /SDA -> /ESP_TXD
- J4 pad 4: /SCL -> GND
- J5 pad 1: /ESP_EN -> +3V3
- J5 pad 2: +3V3 -> GND
- J5 pad 3: /ESP_TXD -> /BRAKE_SCL
- J5 pad 4: GND -> /BRAKE_PWM
Routing:
- net /ESP_EN: track 22.3 -> 84.3 mm
- net /SCL: track 110.2 -> 53.2 mm, vias 2 -> 0
- net /ESP_IO0: track 103.9 -> 56.0 mm, vias 0 -> 2
- net GND: track 122.0 -> 80.6 mm, vias 31 -> 34
- net /SDA: track 107.2 -> 65.9 mm, vias 4 -> 3
- net /R_RGB: track 52.3 -> 20.5 mm
- net /FDCAN_TX: track 72.9 -> 41.6 mm
- net /ESP_TXD: track 62.7 -> 31.5 mm
- net /B_RGB: track 54.2 -> 25.1 mm
- net /G_RGB: track 40.3 -> 17.2 mm
- net /ESP_RXD: track 57.3 -> 34.2 mm
- net /BRAKE_SCL: track 33.9 -> 54.6 mm
- net +3V3: track 81.4 -> 66.5 mm, vias 15 -> 16
- net /USB_D-: track 15.3 -> 2.72 mm
- net /USB_D+: track 14.6 -> 3.41 mm
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- added copper zone on In1.Cu, net GND
- removed copper zone on In2.Cu, net GND
Other:
- board size 75 x 75 mm -> 50 x 50 mm

Commit message: Almost
Parts:
- moved C17 146.0 mm to (91.0, 183.0)
- moved U8 138.0 mm to (95.0, 175.5)
- moved J10 137.7 mm to (78.4, 160.6), turned to 90 degrees
- moved C15 130.9 mm to (88.6, 155.4)
- moved C16 129.9 mm to (89.4, 167.4)
- moved R1 127.6 mm to (94.0, 143.0)
- moved J9 123.2 mm to (76.4, 144.2), turned to 90 degrees
- moved C5 121.9 mm to (98.0, 145.0), turned to -90 degrees
- moved C7 121.8 mm to (94.0, 145.2), turned to -90 degrees
- moved U9 118.5 mm to (94.0, 158.3)
- moved J6 95.5 mm to (79.4, 177.2), turned to 90 degrees
- moved U3 93.2 mm to (91.0, 144.4)
Routing:
- net +3V3: track 66.5 -> 149.0 mm, vias 16 -> 19
- net GND: track 80.6 -> 161.3 mm
- net /SDA2_TTS: track 23.3 -> 54.0 mm
- net /SCL2_TTS: track 26.1 -> 48.3 mm
- net /SDA: track 65.9 -> 85.8 mm, vias 3 -> 4
- net /BRAKE_PWM: track 49.7 -> 69.2 mm
- net /BRAKE_SCL: track 54.6 -> 73.9 mm
- net /SCL: track 53.2 -> 71.4 mm
- net Net-(U3-XSHUT): track 0.00 -> 10.8 mm, vias 0 -> 2
- net Net-(U7-SW): track 13.7 -> 22.1 mm, vias 0 -> 2
Other:
- board size 50 x 50 mm -> 81 x 50 mm

Commit message: FINALLY DONE
Parts:
- removed C15, C17, C5, C6: 100nF, Capacitor_SMD:C_0402_1005Metric_Pad0.74x0.62mm_HandSolder
- removed C16: 10uF, Capacitor_SMD:C_0603_1608Metric
- removed C7: 4U7, Capacitor_SMD:C_0603_1608Metric
- removed J10, J6, J9: 430450400, sensors:CONN_SD-43045-001_04_MOL
- removed J3: Conn_01x04, Connector_JST:JST_SH_SM04B-SRSS-TB_1x04-1MP_P1.00mm_Horizontal
- removed J4: Conn_02x03_Odd_Even, Connector_PinHeader_2.54mm:PinHeader_2x03_P2.54mm_Vertical
- removed R1: 10K, Resistor_SMD:R_0402_1005Metric_Pad0.72x0.64mm_HandSolder
- removed R2, R3: 5k1, Resistor_SMD:R_0402_1005Metric_Pad0.72x0.64mm_HandSolder
- removed U3: VL53L0CXV0DH_1, sensors:XDCR_VL53L0CXV0DH_1
- removed U8: MLX90614ESF-BCF-000-TU, sensors:MLX90614xCF_MEL
- removed U9: MLX90641ESF-BCB-000-TU, sensors:MLX90614xCF_MEL
- added C18: 10uF, Capacitor_SMD:C_0603_1608Metric, F.Cu at (45.9, -18.5)
- added G***: LOGO, LOGO, F.Cu at (-109.0, 29.7)
- added G***: LOGO, LOGO, B.Cu at (29.8, -55.1)
- added G***: LOGO, LOGO, B.Cu at (30.7, -31.7)
- added H1: MountingHole, MountingHole:MountingHole_4.3mm_M4, F.Cu at (62.8, -0.36)
- added H2: MountingHole, MountingHole:MountingHole_4.3mm_M4, F.Cu at (62.8, -64.5)
- added H3: MountingHole, MountingHole:MountingHole_4.3mm_M4, F.Cu at (-1.24, -64.5)
- added H4: MountingHole, MountingHole:MountingHole_4.3mm_M4, F.Cu at (-1.24, -0.36)
- added R19: 470K, Resistor_SMD:R_0603_1608Metric_Pad0.98x0.95mm_HandSolder, F.Cu at (45.8, -12.6)
- added SW3: SW_Wuerth_450301014042, Button_Switch_THT:SW_Slide-03_Wuerth-WS-SLTV_10x2.5x6.4_P2.54mm, F.Cu at (52.4, 2.41)
- added U11: LM73100RPWR, sensors:IC_LM73100RPWR, F.Cu at (45.7, -6.95)
- C10, C12, C4: footprint Capacitor_SMD:C_0402_1005Metric_Pad0.74x0.62mm_HandSolder -> Capacitor_SMD:C_0603_1608Metric_Pad1.08x0.95mm_HandSolder
- J1: footprint Connector_USB:USB_C_Receptacle_HRO_TYPE-C-31-M-12 -> Connector_USB:USB_C_Receptacle_GCT_USB4105-xx-A_16P_TopMnt_Horizontal
- R10, R11, R12, R13, R14, R15, R16, R4, R5, R7, R8, R9: footprint Resistor_SMD:R_0402_1005Metric_Pad0.72x0.64mm_HandSolder -> Resistor_SMD:R_0603_1608Metric_Pad0.98x0.95mm_HandSolder
- R18: value 100R -> 100K
- moved R5 249.8 mm to (4.92, -62.9)
- moved D3 245.7 mm to (12.1, -59.4), turned to 90 degrees
- moved C8 245.6 mm to (4.85, -58.6), turned to -90 degrees
- moved SW1 245.0 mm to (-2.57, -57.6)
- moved J5 211.9 mm to (58.1, -35.1), turned to 90 degrees
- moved D1 207.9 mm to (26.5, -21.3)
- moved C9 206.7 mm to (9.26, -67.6)
- moved C10 206.2 mm to (14.7, -67.5)
- moved R10 205.9 mm to (17.3, -54.6)
- moved R4 205.8 mm to (34.4, -20.0)
- moved U6 205.7 mm to (32.7, -63.3)
- moved U4 204.1 mm to (6.13, -48.8)
- moved R11 203.6 mm to (24.9, -44.9)
- moved J1 203.5 mm to (-3.86, -48.4)
- moved R12 203.4 mm to (29.4, -44.8)
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Connections:
- C13 pad 1: Net-(C13-Pad1) -> +5V
- C14 pad 1: Net-(C13-Pad1) -> +5V
- J1 pad A5: /CC1 -> unconnected-(J1-CC1-PadA5)
- J1 pad B5: /CC2 -> unconnected-(J1-CC2-PadB5)
- R17 pad 2: /CANH -> Net-(SW3-B)
- R18 pad 1: Net-(U7-FB) -> +5V
- R18 pad 2: Net-(C13-Pad1) -> Net-(U7-FB)
- U5 pad 7: unconnected-(U5-Vcc-Pad7) -> Net-(U11-OUT)
- U5 pad 8: unconnected-(U5-Vcc-Pad8) -> Net-(U11-OUT)
- U6 pad 31: /FDCAN_TX -> /FDCAN_RX
- U6 pad 32: /FDCAN_RX -> /FDCAN_TX
- U6 pad 36: /ESP_RXD -> unconnected-(U6-RXD0-Pad36)
- U6 pad 37: /ESP_TXD -> unconnected-(U6-TXD0-Pad37)
Routing:
- net /G_RGB: track 17.2 -> 113.4 mm
- net GND: track 161.3 -> 77.7 mm, vias 34 -> 27
- net +3V3: track 149.0 -> 68.3 mm, vias 19 -> 12
- net /R_RGB: track 20.5 -> 78.3 mm
- net /ESP_EN: track 84.3 -> 32.7 mm, vias 2 -> 0
- net /BRAKE_SCL: track 73.9 -> 28.9 mm, vias 1 -> 0
- net +12V: track 24.8 -> 62.3 mm
- net /ESP_RXD: track 34.2 -> 0.00 mm, vias 2 -> 0
- net +5V: track 91.7 -> 125.0 mm, vias 5 -> 4
- net /ESP_TXD: track 31.5 -> 0.00 mm, vias 2 -> 0
- net /SDA: track 85.8 -> 58.1 mm, vias 4 -> 3
- net /SCL: track 71.4 -> 45.2 mm
- net /BRAKE_PWM: track 69.2 -> 43.0 mm, vias 1 -> 0
- net /CANH: track 7.42 -> 29.3 mm
- net /B_RGB: track 25.1 -> 46.8 mm
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- removed copper zone on B.Cu, net GND
- removed copper zone on F.Cu, net GND
Other:
- board size 81 x 50 mm -> 75 x 75 mm
- board text added: "By: Rayhan Ebrahim"
- board text added: "Onboarding DAQ"
