File: _restore_backup_2026-08-21T02-36-13-544/onboarding.kicad_sch (KiCad schematic)
At the start: 62 parts, among them J1 USB_C_Receptacle_USB2.0_16P, J11 430450800, J12 430450800, J13 430450800, J14 430450800, J15 430450800, J16 430450800, J2 430450800, J4 Conn_01x04, J5 Conn_02x03_Odd_Even, SW1 RESET, SW2 BOOT, U1 LM1117DT-3.3, U10 TJA1462ATK_0Z, U2 ASM330LHHXTR, U3 VL53L0CXV0DH_1, U4 USBLC6-2SC6, U5 STEF12SAGR, U6 ESP32-S3-WROOM-1, U7 LMR51420YFDDCR, U8 MLX90614ESF-BCF-000-TU, U9 MLX90641ESF-BCB-000-TU

Commit message: Maybe I can get this done
Parts:
- removed J11, J12, J13, J14, J15, J16: 430450800, sensors:CONN_SD-43045-001_08_MOL, symbol 430450800:430450800
- added J3: 430450800, sensors:CONN_SD-43045-001_08_MOL, symbol 430450800:430450800
- added J6, J7: 430451600, sensors:CONN_SD-43045-001_16_MOL, symbol 430451600:430451600
- U9: footprint sensors:MLX90614xCF_MEL -> sensors:TO254P912H435-4
Connections:
- net +12V: now also J3.1, J3.2; no longer C11.1, U5.5 (Source), U5.6 (Source), U7.3 (VIN), U7.5 (EN)
- net +3V3: now also R12.2, R13.2, J6.1, J6.2, J7.1, J7.2; no longer R12.1, R13.1
- net BRAKE_PWM: now also J6.15, J6.16, J7.15, J7.16
- net BRAKE_SCL: now also J6.13, J6.14, J7.13, J7.14; no longer U6.21 (IO13), U8.1 (SCL/Vz)
- net CANH: now also J2.7, J2.8, J3.7, J3.8; no longer J2.5, J2.6
- net CANL: now also J2.5, J2.6, J3.5, J3.6; no longer J2.7, J2.8
- net D+: now also U4.4 (I/O2); no longer U4.6 (I/O1)
- net D-: now also U4.6 (I/O1); no longer U4.4 (I/O2)
- net FDCAN_RX: now also U10.1 (TXD); no longer U10.4 (RXD)
- net FDCAN_TX: now also U10.4 (RXD); no longer U10.1 (TXD)
- net GND: now also J3.3, J3.4, J6.3, J6.4, J7.3, J7.4
- net SCL: now also J6.7, J6.8, J7.7, J7.8; no longer R11.2, U6.17 (IO9)
- net SCL2_TTS: now also R12.1, J6.10, J6.9, J7.10, J7.9; no longer R12.2
- net SDA: now also J6.5, J6.6, J7.5, J7.6
- net SDA2_TTS: now also R13.1, J6.11, J6.12, J7.11, J7.12; no longer R13.2
- new net 12 V POST FUSE: C11.1, U5.5 (Source), U5.6 (Source), U7.3 (VIN), U7.5 (EN)
- new net BRAKE_SCL_DBG: U6.21 (IO13), U8.1 (SCL/Vz)
- new net SLC: R11.2, U6.17 (IO9)
Other:
- note removed: "Brake Temp Sensor Connector"
- note removed: "Ride Height Sensor Connector"
- note removed: "Tire Temp Sensor Connector"
