File: _restore_backup_2026-08-22T13-02-49-992/onboarding.kicad_sch (KiCad schematic)
At the start: 62 parts, among them J1 USB_C_Receptacle_USB2.0_16P, J10 430450400, J2 430450800, J3 Conn_01x04, J4 Conn_02x03_Odd_Even, J5 430450400, J6 430450400, J7 430450400, J8 430450400, J9 430450400, SW1 RESET, SW2 BOOT, U1 LM1117DT-3.3, U10 TJA1462ATK_0Z, U2 ASM330LHHXTR, U3 VL53L0CXV0DH_1, U4 USBLC6-2SC6, U5 STEF12SAGR, U6 ESP32-S3-WROOM-1, U7 LMR51420YFDDCR, U8 MLX90614ESF-BCF-000-TU, U9 MLX90641ESF-BCB-000-TU

Commit message: The end is inevitable
Parts:
- removed J10, J5, J6, J9: 430450400, CONN_SD-43045-001_04_MOL, symbol 2026-08-22_02-57-53:430450400
- removed J7, J8: 430450400, sensors:CONN_SD-43045-001_04_MOL, symbol 2026-08-22_02-57-53:430450400
- added J11, J12, J13, J14, J15, J16: 430450800, sensors:CONN_SD-43045-001_08_MOL, symbol 430450800:430450800
- J1: footprint Connector_USB:USB_C_Receptacle_HRO_TYPE-C-31-M-12 -> Connector_USB:USB_C_Receptacle_HCTL_HC-TYPE-C-16P-01A
- renumbered J3 to J4, J4 to J5
Connections:
- net +3V3: now also J11.1, J11.2, J12.1, J12.2, J13.1, J13.2, J14.1, J14.2, J15.1, J15.2, J16.1, J16.2
- net BRAKE_PWM: now also J13.7, J13.8, J16.7, J16.8
- net BRAKE_SCL: now also J13.5, J13.6, J16.5, J16.6
- net GND: now also J11.3, J11.4, J12.3, J12.4, J13.3, J13.4, J14.3, J14.4, J15.3, J15.4, J16.3, J16.4
- net SCL: now also J11.7, J11.8, J14.7, J14.8
- net SCL2_TTS: now also J12.5, J12.6, J15.5, J15.6
- net SDA: now also J11.5, J11.6, J14.5, J14.6
- net SDA2_TTS: now also J12.7, J12.8, J15.7, J15.8
